Commit message: Integrate v2 flange and full gripper collision description

File: ros2_ws/src/atom_gripper_description/urdf/atom_gripper.urdf.xacro (robot description, xacro)
@@ -34,6 +34,7 @@
       </visual>
       <collision>
-        <origin xyz="0 0 0.055"/>
-        <geometry><box size="0.120 0.105 0.110"/></geometry>
+        <!-- Full inherited mesh AABB + 0.5 mm per side; CAD-only envelope. -->
+        <origin xyz="-0.004999999 -0.000000002 0.051335998"/>
+        <geometry><box size="0.131000004 0.106000000 0.118399998"/></geometry>
       </collision>
     </link>
@@ -52,7 +53,7 @@
       </visual>
       <collision>
-        <!-- Box aligned to the visible terminal pad in the transformed CAD mesh. -->
-        <origin xyz="0.021 0.0005 0.154"/>
-        <geometry><box size="0.006 0.020 0.020"/></geometry>
+        <!-- Full inherited mesh AABB + 0.5 mm per side; CAD-only envelope. -->
+        <origin xyz="0.005528131 0.000499999 0.115035999"/>
+        <geometry><box size="0.073943745 0.062999999 0.106999996"/></geometry>
       </collision>
     </link>
@@ -74,7 +75,7 @@
       </visual>
       <collision>
-        <!-- Box aligned to the visible terminal pad in the transformed CAD mesh. -->
-        <origin xyz="-0.024681 0.00045 0.154"/>
-        <geometry><box size="0.006 0.020 0.020"/></geometry>
+        <!-- Full inherited mesh AABB + 0.5 mm per side; CAD-only envelope. -->
+        <origin xyz="-0.009208677 0.000450000 0.115035999"/>
+        <geometry><box size="0.073943744 0.062999999 0.106999996"/></geometry>
       </collision>
     </link>

File: ros2_ws/src/atom_xarm_description/urdf/uf850_atom.urdf.xacro (robot description, xacro)
@@ -19,7 +19,7 @@
     create_attach_link="true"
     load_gazebo_plugin="false"/>
-  <xacro:include filename="$(find atom_gripper_description)/urdf/atom_gripper.urdf.xacro"/>
-  <xacro:atom_gripper parent="$(arg prefix)link_eef" prefix="$(arg prefix)" use_mimic="true">
+  <xacro:include filename="$(find atom_gripper_description)/urdf/atom_gripper_v2.urdf.xacro"/>
+  <xacro:atom_gripper_v2 parent="$(arg prefix)link_eef" prefix="$(arg prefix)">
     <origin xyz="$(arg gripper_mount_xyz)" rpy="$(arg gripper_mount_rpy)"/>
-  </xacro:atom_gripper>
+  </xacro:atom_gripper_v2>
 </robot>
