Commit message: Integrate mobile base, refresh hardware assets, and add A4 tag print sheets

File: ros2_ws/src/atom_gripper_description/urdf/atom_mount_v2.urdf.xacro (robot description, xacro)
@@ -1,27 +1,34 @@
 <?xml version="1.0"?>
 <robot xmlns:xacro="http://www.ros.org/wiki/xacro">
-  <!-- CAD-only placement; no measured mass/CoM. Not a dynamics model. -->
+  <!-- Nominal CAD review only; inertial and camera calibration are unmeasured. -->
   <xacro:macro name="atom_mount_v2" params="parent gripper_base prefix:=''">
-    <link name="${prefix}camera_bracket">
-      <visual><origin xyz="-0.043494000 -0.022225000 0.028836000" rpy="1.5707963267948966 1.5707963267948966 0"/>
-        <geometry><mesh filename="package://atom_gripper_description/meshes/generated/mount_v2/camera_bracket.stl" scale="0.001 0.001 0.001"/></geometry>
+    <link name="${prefix}flange_adapter">
+      <visual><origin xyz="-0.043494000 -0.022225000 0.080800000" rpy="1.5707963267948966 1.5707963267948966 0"/>
+        <geometry><mesh filename="package://atom_gripper_description/meshes/generated/mount/flange_adapter.stl" scale="0.001 0.001 0.001"/></geometry>
         <material name="atom_mount"><color rgba="0.25 0.45 0.65 1"/></material></visual>
-      <collision><origin xyz="0.000000000 -0.048550000 0.075036000"/><geometry><box size="0.019000000 0.018900000 0.071000000"/></geometry></collision>
+      <collision><origin xyz="0.000000000 -0.000000000 0.025000000"/><geometry><box size="0.085000000 0.113000000 0.055000000"/></geometry></collision>
     </link>
-    <joint name="${prefix}camera_bracket_joint" type="fixed"><parent link="${gripper_base}"/><child link="${prefix}camera_bracket"/></joint>
+    <joint name="${prefix}flange_adapter_joint" type="fixed"><parent link="${parent}"/><child link="${prefix}flange_adapter"/></joint>
     <link name="${prefix}esp32_bracket">
       <visual><origin xyz="-0.043494000 -0.022225000 0.028836000" rpy="1.5707963267948966 1.5707963267948966 0"/>
-        <geometry><mesh filename="package://atom_gripper_description/meshes/generated/mount_v2/esp32_bracket.stl" scale="0.001 0.001 0.001"/></geometry>
+        <geometry><mesh filename="package://atom_gripper_description/meshes/generated/mount/esp32_bracket.stl" scale="0.001 0.001 0.001"/></geometry>
         <material name="atom_mount"><color rgba="0.25 0.45 0.65 1"/></material></visual>
       <collision><origin xyz="0.000000000 0.048550000 0.073536000"/><geometry><box size="0.043000000 0.018900000 0.068000000"/></geometry></collision>
     </link>
     <joint name="${prefix}esp32_bracket_joint" type="fixed"><parent link="${gripper_base}"/><child link="${prefix}esp32_bracket"/></joint>
-    <link name="${prefix}flange_adapter">
-      <visual><origin xyz="-0.043494000 -0.022225000 0.080800000" rpy="1.5707963267948966 1.5707963267948966 0"/>
-        <geometry><mesh filename="package://atom_gripper_description/meshes/generated/mount_v2/flange_adapter.stl" scale="0.001 0.001 0.001"/></geometry>
+    <link name="${prefix}camera_bracket">
+      <visual><origin xyz="-0.043494000 -0.022225000 0.028836000" rpy="1.5707963267948966 1.5707963267948966 0"/>
+        <geometry><mesh filename="package://atom_gripper_description/meshes/generated/mount/camera_bracket.stl" scale="0.001 0.001 0.001"/></geometry>
         <material name="atom_mount"><color rgba="0.25 0.45 0.65 1"/></material></visual>
-      <collision><origin xyz="0.000000000 -0.000000000 0.025000000"/><geometry><box size="0.085000000 0.113000000 0.055000000"/></geometry></collision>
+      <collision><origin xyz="0.000000000 -0.064049999 0.062536000"/><geometry><box size="0.066000000 0.049900002 0.046000000"/></geometry></collision>
     </link>
-    <joint name="${prefix}flange_adapter_joint" type="fixed"><parent link="${parent}"/><child link="${prefix}flange_adapter"/></joint>
+    <joint name="${prefix}camera_bracket_joint" type="fixed"><parent link="${gripper_base}"/><child link="${prefix}camera_bracket"/></joint>
+    <!-- Nominal D435i housing; USB/cables/optical TF and inertial data absent. -->
+    <link name="${prefix}d435i_body">
+      <visual><geometry><box size="0.090000000 0.025000000 0.025050000"/></geometry>
+        <material name="atom_camera"><color rgba="0.55 0.57 0.60 1"/></material></visual>
+      <collision><origin xyz="0 0 0"/><geometry><box size="0.091000000 0.026000000 0.026050000"/></geometry></collision>
+    </link>
+    <joint name="${prefix}d435i_body_joint" type="fixed"><parent link="${gripper_base}"/><child link="${prefix}d435i_body"/><origin xyz="0.000000000 -0.073000000 0.097561000" rpy="0 0 0"/></joint>
   </xacro:macro>
 </robot>

File: ros2_ws/src/atom_xarm_description/srdf/uf850_atom.srdf.xacro (robot description, xacro)
@@ -14,4 +14,5 @@
     <link name="$(arg prefix)camera_bracket"/>
     <link name="$(arg prefix)esp32_bracket"/>
+    <link name="$(arg prefix)d435i_body"/>
   </group>
   <end_effector name="$(arg prefix)atom_tool" parent_link="$(arg prefix)link_eef" group="$(arg prefix)atom_tool" parent_group="$(arg prefix)uf850"/>
@@ -34,4 +35,6 @@
   <disable_collisions link1="$(arg prefix)flange_adapter" link2="$(arg prefix)esp32_bracket" reason="ToolEnvelopeOverlap"/>
   <disable_collisions link1="$(arg prefix)camera_bracket" link2="$(arg prefix)esp32_bracket" reason="ToolEnvelopeOverlap"/>
+  <!-- Camera housing/bracket mounting contact only; camera vs fingers/arm stays checked. -->
+  <disable_collisions link1="$(arg prefix)d435i_body" link2="$(arg prefix)camera_bracket" reason="CameraMountContact"/>
   <!-- Only adapter/flange mounting contact is excluded against the arm. -->
   <disable_collisions link1="$(arg prefix)flange_adapter" link2="$(arg prefix)link6" reason="FlangeMountContact"/>

File: ros2_ws/src/atom_xarm_description/urdf/uf850_atom.urdf.xacro (robot description, xacro)
@@ -2,4 +2,7 @@
 <robot xmlns:xacro="http://ros.org/wiki/xacro" name="ATOM_UF850">
   <xacro:arg name="prefix" default=""/>
+  <!-- Offline review uses fake hardware; deployment must explicitly select a verified driver/IP. -->
+  <xacro:arg name="ros2_control_plugin" default="fake_components/GenericSystem"/>
+  <xacro:arg name="robot_ip" default=""/>
   <xacro:arg name="gripper_mount_xyz" default="0 0 0"/>
   <xacro:arg name="gripper_mount_rpy" default="0 0 0"/>
@@ -8,4 +11,6 @@
     prefix="$(arg prefix)"
     hw_ns="ufactory"
+    ros2_control_plugin="$(arg ros2_control_plugin)"
+    robot_ip="$(arg robot_ip)"
     limited="true"
     dof="6"
